Commit message: opg 1 ferdig

File: src/qube_description/urdf/qube.macro.xacro (robot description, xacro)
@@ -13,4 +13,5 @@
     <xacro:property name="ind_x" value="${ind_l/2.0}"/>
     <xacro:property name="ind_z" value="${rotor_half + ind_h/2.0}"/>
+    <link name="${prefix}base_link"/>
     <link name="${prefix}stator_link">
       <visual>

File: src/qube_description/urdf/qube.urdf.xacro (robot description, xacro)
@@ -1,4 +1,4 @@
 <?xml version="1.0"?>
-<robot xmlns:xacro="http://www.ros.org/wiki/xacro">
+<robot name="qube" xmlns:xacro="http://www.ros.org/wiki/xacro">
   <!-- Inkluder makrofilen -->
   <xacro:include filename="$(find qube_description)/urdf/qube.macro.xacro"/>
@@ -6,5 +6,5 @@
   <link name="world"/>
   <!-- Kall qube-makroen -->
-  <xacro:qube/>
+  <xacro:qube prefix=""/>
   <!-- Koble world til base_link -->
   <joint name="world_to_base" type="fixed">
